File: KiCad/Patchworks.kicad_sch (KiCad schematic)
At the start: 52 parts, among them J1 VEE Bolt, J10 5V Bus, J11 3V3 Bus, J12 DC, J2 VIN Bolt (4-40VDC), J3 GND Bolt, J4 3V3 Bus, J5 5V Bus, J6 5V Bus, J7 VCC Bus, J8 VCC Bus, J9 5V Bus, K1 Relay, M1 5V, Q1 2N3904, Q2 2N3904, SW1 Post, SW2 Power On, U1 LM317 Regulator (VCC 5-12VDC), U2 Power Monitor, U3 LCD Display, U4 BB Power, U5 PIC16F887-IP, Y1 4MHz

Commit message: Rename repo
Other:
- title: Board -> Patchworks
Changed lines of the file:
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@@
 	(paper "USLetter")
 	(title_block
-		(title "Board")
+		(title "Patchworks")
 		(date "2024-04-15")
 		(rev "1")
